File: docs/KiCad - TTF 240х240/Дисплей 240х240.kicad_pcb (KiCad board)
At the start: 2 copper layers, 37 x 38.2 mm, 42 parts, among them J1 Display, J2 USB, J3 Input, Q1 AO3402, SW1 reset, SW2 boot, U1 SN65HVD230, U2 THVD1406D, U3 LMR50410, U5 ESP32-C3-MINI-1U, U7 AP2112K-3.3

Commit message: Редактирование схемы и пп
Connections:
- net +4V renamed /+4V
